File: Valve Wizard Cab Sim.kicad_sch (KiCad schematic)
At the start: 54 parts, among them J1 IN, J10 IN, J11 IN, J2 FS, J3 Power, J4 Battery, J5 FS_F, J6 GND, J7 FS, J8 FS_E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

Commit message: latest
Parts:
- removed J2, J7: FS, Connector_PinHeader_2.54mm:PinHeader_1x01_P2.54mm_Vertical, symbol Connector:Conn_01x01_Female
- removed J5: FS_F, Connector_PinHeader_2.54mm:PinHeader_1x01_P2.54mm_Vertical, symbol Connector:Conn_01x01_Female
- removed J8: FS_E, Connector_PinHeader_2.54mm:PinHeader_1x01_P2.54mm_Vertical, symbol Connector:Conn_01x01_Female
- removed Q1: MMDT3946, Package_TO_SOT_SMD:SOT-363_SC-70-6, symbol Transistor_BJT:MMDT3946
- added #J7: AudioPlug3, symbol Connector:AudioPlug3
- added J2: FS_EF, Wire_Connector_Supported:PinHeader_1x02_P2.54mm_Vertical, symbol Connector:Conn_01x02_Female
- added J5: FS, Wire_Connector_Supported:PinHeader_1x02_P2.54mm_Vertical, symbol Connector:Conn_01x02_Female
- added Q2: BC846BPN, Package_TO_SOT_SMD:SOT-363_SC-70-6, symbol Transistor_BJT:BC846BPN
- C1, C11: footprint Capacitor_Tantalum_SMD:CP_EIA-7343-43_Kemet-X_Pad2.25x2.55mm_HandSolder -> Capacitor_THT:CP_Radial_D10.0mm_P5.00mm; LCSC C600572 -> (none)
- J1, J4, J6: footprint Connector_PinHeader_2.54mm:PinHeader_1x02_P2.54mm_Vertical -> Wire_Connector_Supported:PinHeader_1x02_P2.54mm_Vertical
- J10: footprint Connector_Audio:Jack_6.35mm_Neutrik_NMJ6HCD2_Horizontal -> MyLibraries:Jack_6.35mm_Neutrik_NMJ6HC-S_SOLDER_LUG; symbol Connector:AudioJack3_Ground_Switch -> Connector:AudioJack3_Switch
- J11: value IN -> OUT; footprint Connector_Audio:Jack_6.35mm_Neutrik_NMJ6HCD2_Horizontal -> MyLibraries:Jack_6.35mm_Neutrik_NMJ6HC-S_SOLDER_LUG; symbol Connector:AudioJack3_Ground_Switch -> Connector:AudioJack3_Switch
- R7: LibPart (none) -> C17902
- RV1, RV2: symbol Device:R_Potentiometer_Small -> Device:R_Potentiometer_MountingPin
- U1: LCSC (none) -> C6961
Connections:
- net +9V: now also Q2.6 (C1)
- net FS_A: now also J5.2 (Pin_2)
- net FS_CD: now also #J7.T, J5.1 (Pin_1)
- net FS_E: now also J2.2 (Pin_2)
- net FS_F: now also J2.1 (Pin_1)
- net GND: now also J10.RN, J10.SN, J11.RN, J11.SN, J11.TN, RV1.MP (MountPin), RV2.MP (MountPin), #J7.R, Q2.3 (C2)
- net at R15.1, R16.2, U1.6 (-): now also Q2.1 (E1), Q2.4 (E2)
- net at R15.2, U1.7: now also Q2.2 (B1), Q2.5 (B2)
- net Sleeve: now reaches C12.1, J11.S
- net Sleeve: now also #J7.S
- no-connect marks 7 -> 0
Other:
- moved on the sheet: C12, J6
